File: motionControl.sch (KiCad schematic (older format))
At the start: 42 parts, among them U301 TMC4671-ES, U302 SN74LVC3G17DCURE4, U303 SN74LVC3G17DCURE4, Y301 MC2016K25.0000C16ESH

Commit message: ultima actualizacion antes de iniciar el ruteado, diseño verificado
Parts:
- added C325, C326: 1uF/50V/0805, Capacitor_SMD:C_0805_2012Metric, symbol Device:C
- added J301, J302: Conn_01x05, Connector_PinHeader_2.54mm:PinHeader_1x05_P2.54mm_Vertical, symbol Connector_Generic:Conn_01x05
- U301: symbol TMC4671-ES:TMC4671-ES -> spincoater-rescue:TMC4671-ES-TMC4671-ES
Connections:
- net labels added: SPI_SCK
- net labels removed: BRAKE_4671, ENC1_A, ENC1_B, ENC1_N, HALL_UX, HALL_V, HALL_WY, SPI_CLK, STATUS_4671
- wire segments 141 -> 159
- no-connect marks 29 -> 31
Other:
- moved on the sheet: C307, C308, C309, C310, C311, C312, C313, C314, C315
