File: driverMotor.sch (KiCad schematic (older format))
At the start: 43 parts, among them Q401 SI7288DP-T1-GE3, Q402 SI7288DP-T1-GE3, Q403 SI7288DP-T1-GE3, U401 AD8418-Amplifier_Current, U402 TMC6100-LA, U403 AD8418-Amplifier_Current

Commit message: ultima actualizacion antes de iniciar el ruteado, diseño verificado
Parts:
- added J401: 1803280, 1803280:1803280, symbol ConnectorX3:1803280
Connections:
- net U: no longer C420.1
- net V: no longer C421.1
- net W: no longer C422.1
- net at L401.2: now also C420.1, J401.1
- net at L402.2: now also C421.1, J401.2
- net at L403.2: now also C422.1, J401.3
- net FAULT_6100: no longer names the net of U402.23 (FAULT)
- no-connect marks 2 -> 3
Other:
- moved on the sheet: C420, C421, C422, L401, L402, L403
Changed lines of the file:
@@
 	2150 6300 2150 5800
 Connection ~ 2150 6300
-Text Label 2150 5800 0    50   ~ 0
-+2.5V_REF
-Text Label 5050 5800 0    50   ~ 0
-+2.5V_REF
 $Comp
 L Device:R R404
@@
 	5700 3550 5650 3550
 $Comp
-L Device:C C408
-U 1 1 5EE57627
-P 4150 1250
-F 0 "C408" V 3898 1250 50  0000 C CNN
-F 1 "100nF/50V/0603" V 3989 1250 50  0000 C CNN
-F 2 "Capacitor_SMD:C_0603_1608Metric" H 4188 1100 50  0001 C CNN
-F 3 "~" H 4150 1250 50  0001 C CNN
-	1    4150 1250
-	0    1    1    0
-$EndComp
-$Comp
 L Device:C C410
 U 1 1 5EE577EF
@@
 	1    0    0    -1
 $EndComp
-Wire Wire Line
-	4000 1250 3950 1250
-Wire Wire Line
-	3950 1250 3950 1350
 Wire Wire Line
 	4300 1250 4350 1250
@@
 Wire Wire Line
 	2950 2450 2850 2450
-Text Label 1850 2600 2    50   ~ 0
-CS_6100
-Text Label 2950 2700 2    50   ~ 0
-SPI_SCK
-Text Label 2950 2800 2    50   ~ 0
-SPI_MOSI
-Text Label 2950 2900 2    50   ~ 0
-SPI_MISO
-Text Label 2950 3150 2    50   ~ 0
-UH
-Text Label 2950 3250 2    50   ~ 0
-UL
-Text Label 2950 3350 2    50   ~ 0
-VH
-Text Label 2950 3450 2    50   ~ 0
-VL
-Text Label 2950 3550 2    50   ~ 0
-WH
-Text Label 2950 3650 2    50   ~ 0
-WL
 Wire Wire Line
 	2950 3800 2350 3800
@@
 	2350 3800 2350 3750
 Connection ~ 2350 3800
-Text Label 5150 3800 0    50   ~ 0
-FAULT_6100
 Text Label 5900 3000 0    50   ~ 0
 HSW
@@
 	5500 6050 5600 6050
 Connection ~ 5500 6050
-Text Label 2700 6050 0    50   ~ 0
-CUR_U
 Wire Wire Line
 	2550 6050 2700 6050
-Text Label 5600 6050 0    50   ~ 0
-CUR_W
 $Comp
 L power:+24V #PWR0419
@@
 $EndComp
 Connection ~ 4350 1000
-Text Label 2750 2000 0    50   ~ 0
-EN_6100
 $Comp
 L power:+3.3V #PWR0406
@@
 Wire Wire Line
 	1850 2600 2250 2600
-Wire Wire Line
-	2750 2050 2750 2000
 Connection ~ 2750 2050
 Wire Wire Line
@@
 $EndComp
 Connection ~ 3800 6450
-Wire Notes Line
-	6450 5900 10100 5900
-Wire Notes Line
-	10100 750  6450 750
-Wire Notes Line
-	6450 5900 6450 750
 Text Notes 6450 650  0    50   ~ 0
 Driver Stage
@@
 Wire Notes Line
 	550  5650 5900 5650
-Wire Wire Line
-	6950 1000 8200 1000
 Connection ~ 8200 1000
 Wire Wire Line
@@
 L Device:L L401
 U 1 1 5EFC30B4
-P 9650 1550
-F 0 "L401" V 9840 1550 50  0000 C CNN
-F 1 "50R/12A/1206" V 9749 1550 50  0000 C CNN
-F 2 "Inductor_SMD:L_1206_3216Metric" H 9650 1550 50  0001 C CNN
-F 3 "~" H 9650 1550 50  0001 C CNN
-	1    9650 1550
+P 9300 1550
+F 0 "L401" V 9490 1550 50  0000 C CNN
+F 1 "50R/12A/1206" V 9399 1550 50  0000 C CNN
+F 2 "Inductor_SMD:L_1206_3216Metric" H 9300 1550 50  0001 C CNN
+F 3 "~" H 9300 1550 50  0001 C CNN
+	1    9300 1550
 	0    -1   -1   0
 $EndComp
@@
 L Device:C C420
 U 1 1 5EFC3B7E
-P 9350 1800
-F 0 "C420" H 9250 1900 50  0000 L CNN
-F 1 "1nF/100V/0603" V 9200 1300 50  0000 L CNN
-F 2 "Capacitor_SMD:C_0603_1608Metric" H 9388 1650 50  0001 C CNN
-F 3 "~" H 9350 1800 50  0001 C CNN
-	1    9350 1800
-	1    0    0    -1
-$EndComp
-Wire Wire Line
-	8750 1550 9350 1550
-Wire Wire Line
-	9350 1650 9350 1550
-Connection ~ 9350 1550
+P 9650 1850
+F 0 "C420" H 9550 1950 50  0000 L CNN
+F 1 "1nF/100V/0603" V 9500 1350 50  0000 L CNN
+F 2 "Capacitor_SMD:C_0603_1608Metric" H 9688 1700 50  0001 C CNN
+F 3 "~" H 9650 1850 50  0001 C CNN
+	1    9650 1850
+	1    0    0    -1
+$EndComp
 $Comp
 L power:GND #PWR0434
 U 1 1 5EFCB46D
-P 9350 2150
-F 0 "#PWR0434" H 9350 1900 50  0001 C CNN
-F 1 "GND" H 9355 1977 50  0000 C CNN
-F 2 "" H 9350 2150 50  0001 C CNN
-F 3 "" H 9350 2150 50  0001 C CNN
-	1    9350 2150
-	1    0    0    -1
-$EndComp
-Wire Wire Line
-	9350 1950 9350 2150
+P 9650 2200
+F 0 "#PWR0434" H 9650 1950 50  0001 C CNN
+F 1 "GND" H 9655 2027 50  0000 C CNN
+F 2 "" H 9650 2200 50  0001 C CNN
+F 3 "" H 9650 2200 50  0001 C CNN
+	1    9650 2200
+	1    0    0    -1
+$EndComp
+Wire Wire Line
+	9650 2000 9650 2200
 $Comp
 L Device:C C421
 U 1 1 5EFD9D2A
-P 9350 3600
-F 0 "C421" H 9250 3700 50  0000 L CNN
-F 1 "1nF/100V/0603" V 9200 3100 50  0000 L CNN
-F 2 "Capacitor_SMD:C_0603_1608Metric" H 9388 3450 50  0001 C CNN
-F 3 "~" H 9350 3600 50  0001 C CNN
-	1    9350 3600
+P 9600 3650
+F 0 "C421" H 9500 3750 50  0000 L CNN
+F 1 "1nF/100V/0603" V 9450 3150 50  0000 L CNN
+F 2 "Capacitor_SMD:C_0603_1608Metric" H 9638 3500 50  0001 C CNN
+F 3 "~" H 9600 3650 50  0001 C CNN
+	1    9600 3650
 	1    0    0    -1
 $EndComp
@@
 L Device:L L402
 U 1 1 5EFDA4D2
-P 9650 3350
-F 0 "L402" V 9840 3350 50  0000 C CNN
-F 1 "50R/12A/1206" V 9749 3350 50  0000 C CNN
-F 2 "Inductor_SMD:L_1206_3216Metric" H 9650 3350 50  0001 C CNN
-F 3 "~" H 9650 3350 50  0001 C CNN
-	1    9650 3350
+P 9300 3350
+F 0 "L402" V 9490 3350 50  0000 C CNN
+F 1 "50R/12A/1206" V 9399 3350 50  0000 C CNN
+F 2 "Inductor_SMD:L_1206_3216Metric" H 9300 3350 50  0001 C CNN
+F 3 "~" H 9300 3350 50  0001 C CNN
+	1    9300 3350
 	0    -1   -1   0
 $EndComp
@@
 L Device:C C422
 U 1 1 5EFE15D1
-P 9350 5350
-F 0 "C422" H 9250 5450 50  0000 L CNN
-F 1 "1nF/100V/0603" V 9200 4850 50  0000 L CNN
-F 2 "Capacitor_SMD:C_0603_1608Metric" H 9388 5200 50  0001 C CNN
-F 3 "~" H 9350 5350 50  0001 C CNN
-	1    9350 5350
+P 9600 5450
+F 0 "C422" H 9500 5550 50  0000 L CNN
+F 1 "1nF/100V/0603" V 9450 4950 50  0000 L CNN
+F 2 "Capacitor_SMD:C_0603_1608Metric" H 9638 5300 50  0001 C CNN
+F 3 "~" H 9600 5450 50  0001 C CNN
+	1    9600 5450
 	1    0    0    -1
 $EndComp
@@
 L Device:L L403
 U 1 1 5EFE1DF7
-P 9650 5150
-F 0 "L403" V 9840 5150 50  0000 C CNN
-F 1 "50R/12A/1206" V 9749 5150 50  0000 C CNN
-F 2 "Inductor_SMD:L_1206_3216Metric" H 9650 5150 50  0001 C CNN
-F 3 "~" H 9650 5150 50  0001 C CNN
-	1    9650 5150
+P 9300 5150
+F 0 "L403" V 9490 5150 50  0000 C CNN
+F 1 "50R/12A/1206" V 9399 5150 50  0000 C CNN
+F 2 "Inductor_SMD:L_1206_3216Metric" H 9300 5150 50  0001 C CNN
+F 3 "~" H 9300 5150 50  0001 C CNN
+	1    9300 5150
 	0    -1   -1   0
 $EndComp
@@
 L power:GND #PWR0436
 U 1 1 5EFE29A7
-P 9350 5650
-F 0 "#PWR0436" H 9350 5400 50  0001 C CNN
-F 1 "GND" H 9355 5477 50  0000 C CNN
-F 2 "" H 9350 5650 50  0001 C CNN
-F 3 "" H 9350 5650 50  0001 C CNN
-	1    9350 5650
+P 9600 5750
+F 0 "#PWR0436" H 9600 5500 50  0001 C CNN
+F 1 "GND" H 9605 5577 50  0000 C CNN
+F 2 "" H 9600 5750 50  0001 C CNN
+F 3 "" H 9600 5750 50  0001 C CNN
+	1    9600 5750
 	1    0    0    -1
 $EndComp
@@
 L power:GND #PWR0435
 U 1 1 5EFE2FA0
-P 9350 3850
-F 0 "#PWR0435" H 9350 3600 50  0001 C CNN
-F 1 "GND" H 9355 3677 50  0000 C CNN
-F 2 "" H 9350 3850 50  0001 C CNN
-F 3 "" H 9350 3850 50  0001 C CNN
-	1    9350 3850
-	1    0    0    -1
-$EndComp
-Wire Wire Line
-	8200 3350 9350 3350
-Wire Wire Line
-	9350 3450 9350 3350
-Connection ~ 9350 3350
-Wire Wire Line
-	9350 3350 9500 3350
-Wire Wire Line
-	9350 3750 9350 3850
-Wire Wire Line
-	9350 1550 9500 1550
-Wire Wire Line
-	8700 5150 9350 5150
-Wire Wire Line
-	9350 5200 9350 5150
-Connection ~ 9350 5150
-Wire Wire Line
-	9350 5150 9500 5150
-Wire Wire Line
-	9350 5500 9350 5650
+P 9600 3900
+F 0 "#PWR0435" H 9600 3650 50  0001 C CNN
+F 1 "GND" H 9605 3727 50  0000 C CNN
+F 2 "" H 9600 3900 50  0001 C CNN
+F 3 "" H 9600 3900 50  0001 C CNN
+	1    9600 3900
+	1    0    0    -1
+$EndComp
+Wire Wire Line
+	9600 3800 9600 3900
+Wire Wire Line
+	9600 5600 9600 5750
+Text GLabel 1850 2600 0    50   Input ~ 0
+CS_6100
+$Comp
+L ConnectorX3:1803280 J401
+U 1 1 5F144E28
+P 10300 3250
+F 0 "J401" H 10350 3550 60  0000 L CNN
+F 1 "1803280" H 10350 3450 60  0000 L CNN
+F 2 "1803280:1803280" H 10700 3090 60  0001 C CNN
+F 3 "" H 10300 3250 60  0000 C CNN
+	1    10300 3250
+	1    0    0    -1
+$EndComp
+Wire Wire Line
+	10050 5150 10050 3450
+Wire Wire Line
+	10050 3450 10300 3450
+Wire Wire Line
+	10050 1550 10050 3250
+Wire Wire Line
+	10050 3250 10300 3250
+Wire Notes Line
+	6450 750  11050 750
+Text GLabel 2950 2700 0    50   Input ~ 0
+SPI_SCK
+Text GLabel 2950 2800 0    50   Input ~ 0
+SPI_MOSI
+Text GLabel 2950 2900 0    50   Input ~ 0
+SPI_MISO
+Text GLabel 2750 1250 0    50   Input ~ 0
+EN_6100
+Text GLabel 2150 5800 2    50   Input ~ 0
++2.5V_REF
+Text GLabel 5050 5800 2    50   Input ~ 0
++2.5V_REF
+Text GLabel 2950 3150 0    50   Input ~ 0
+UH
+Text GLabel 2950 3250 0    50   Input ~ 0
+UL
+Text GLabel 2950 3350 0    50   Input ~ 0
+VH
+Text GLabel 2950 3450 0    50   Input ~ 0
+VL
+Text GLabel 2950 3550 0    50   Input ~ 0
+WH
+Text GLabel 2950 3650 0    50   Input ~ 0
+WL
+Text GLabel 5600 6050 2    50   Input ~ 0
+CUR_W
+Text GLabel 2700 6050 2    50   Input ~ 0
+CUR_U
+$Comp
+L Device:C C408
+U 1 1 5EE57627
+P 4150 1250
+F 0 "C408" V 3898 1250 50  0000 C CNN
+F 1 "100nF/50V/0603" V 3989 1250 50  0000 C CNN
+F 2 "Capacitor_SMD:C_0603_1608Metric" H 4188 1100 50  0001 C CNN
+F 3 "~" H 4150 1250 50  0001 C CNN
+	1    4150 1250
+	0    1    1    0
+$EndComp
+Wire Wire Line
+	4000 1250 3950 1250
+Wire Wire Line
+	3950 1250 3950 1350
+NoConn ~ 5150 3800
+$Comp
+L power:PWR_FLAG #FLG0102
+U 1 1 5F52524C
+P 4850 1000
+F 0 "#FLG0102" H 4850 1075 50  0001 C CNN
+F 1 "PWR_FLAG" H 4850 1173 50  0000 C CNN
+F 2 "" H 4850 1000 50  0001 C CNN
+F 3 "~" H 4850 1000 50  0001 C CNN
+	1    4850 1000
+	1    0    0    -1
+$EndComp
+Connection ~ 4850 1000
+Wire Wire Line
+	6950 1000 8200 1000
+Wire Wire Line
+	2750 1250 2750 2050
+Wire Wire Line
+	8750 1550 9150 1550
+Wire Wire Line
+	9450 1550 9650 1550
+Wire Wire Line
+	9650 1700 9650 1550
+Connection ~ 9650 1550
+Wire Wire Line
+	9650 1550 10050 1550
+Wire Wire Line
+	8200 3350 9150 3350
+Wire Wire Line
+	9450 3350 9600 3350
+Wire Wire Line
+	9600 3500 9600 3350
+Connection ~ 9600 3350
+Wire Wire Line
+	9600 3350 10300 3350
+Wire Wire Line
+	8700 5150 9150 5150
+Wire Wire Line
+	9450 5150 9600 5150
+Wire Wire Line
+	9600 5300 9600 5150
+Connection ~ 9600 5150
+Wire Wire Line
+	9600 5150 10050 5150
+Wire Notes Line
+	6450 6050 11050 6050
+Wire Notes Line
+	6450 750  6450 6050
+Wire Notes Line
+	11050 750  11050 6050
 $EndSCHEMATC

Commit message: antes de comenzar a rutear
Connections:
- net at C420.1, L401.2: now also J401.3; no longer J401.1
- net at C422.1, L403.2: now also J401.1; no longer J401.3
Changed lines of the file:
@@
 L ConnectorX3:1803280 J401
 U 1 1 5F144E28
-P 10300 3250
-F 0 "J401" H 10350 3550 60  0000 L CNN
-F 1 "1803280" H 10350 3450 60  0000 L CNN
-F 2 "1803280:1803280" H 10700 3090 60  0001 C CNN
-F 3 "" H 10300 3250 60  0000 C CNN
-	1    10300 3250
-	1    0    0    -1
+P 10300 3450
+F 0 "J401" H 10350 3750 60  0000 L CNN
+F 1 "1803280" H 10350 3650 60  0000 L CNN
+F 2 "1803280:1803280" H 10700 3290 60  0001 C CNN
+F 3 "" H 10300 3450 60  0000 C CNN
+	1    10300 3450
+	1    0    0    1
 $EndComp
 Wire Wire Line
