File: alimentacion.sch (KiCad schematic (older format))
At the start: 25 parts, among them U501 LP2985-3.3, U502 LMR16020PDDAR

Commit message: ultima actualizacion antes de iniciar el ruteado, diseño verificado
Parts:
- removed D501: D_Schottky_VLS6045, symbol Device:D_Schottky
- added D501: V2PM10HM3, DIODE_MSS1P4-M3:DIODE_MSS1P4-M3, symbol MSS1P4-M3_89A:MSS1P4-M3_89A
- added J501: 1757242, PHOENIX_1757242:PHOENIX_1757242, symbol ConnectorX2:1757242
Connections:
- wire segments 63 -> 71
Other:
- moved on the sheet: C504, C505, C506, C507, C508, C509, L501, L502, R503, R504, R522, U502

Commit message: antes de comenzar a rutear
Parts:
- added D503: SMBJ33A-13-F, SMBJ33A-13-F:SMBJ33A-13-F, symbol SMBJ33A-13-F:SMBJ33A-13-F
Connections:
- net +24V: now also D503.1
- net GND: now also D503.2
Other:
- moved on the sheet: J501
Changed lines of the file:
@@
 Wire Wire Line
 	3900 5750 4150 5750
-Connection ~ 3900 5750
 Wire Notes Line
 	3000 4900 3000 6550
@@
 L ConnectorX2:1757242 J501
 U 1 1 5F121883
-P 1300 1650
-F 0 "J501" H 1193 2017 50  0000 C CNN
-F 1 "1757242" H 1193 1926 50  0000 C CNN
-F 2 "PHOENIX_1757242:PHOENIX_1757242" H 1300 1650 50  0001 L BNN
-F 3 "07/07/2016" H 1300 1650 50  0001 L BNN
-F 4 "Manufacturer Recommendations" H 1300 1650 50  0001 L BNN "Field4"
-F 5 "Phoenix Contact" H 1300 1650 50  0001 L BNN "Field5"
-	1    1300 1650
+P 1000 1650
+F 0 "J501" H 893 2017 50  0000 C CNN
+F 1 "1757242" H 893 1926 50  0000 C CNN
+F 2 "PHOENIX_1757242:PHOENIX_1757242" H 1000 1650 50  0001 L BNN
+F 3 "07/07/2016" H 1000 1650 50  0001 L BNN
+F 4 "Manufacturer Recommendations" H 1000 1650 50  0001 L BNN "Field4"
+F 5 "Phoenix Contact" H 1000 1650 50  0001 L BNN "Field5"
+	1    1000 1650
 	-1   0    0    -1
 $EndComp
@@
 L power:GND #PWR0521
 U 1 1 5F13B1E6
-P 1600 2500
-F 0 "#PWR0521" H 1600 2250 50  0001 C CNN
-F 1 "GND" H 1605 2327 50  0000 C CNN
-F 2 "" H 1600 2500 50  0001 C CNN
-F 3 "" H 1600 2500 50  0001 C CNN
-	1    1600 2500
-	1    0    0    -1
-$EndComp
-Wire Wire Line
-	1600 1550 2050 1550
-Wire Wire Line
-	1600 2500 1600 1750
+P 1300 2450
+F 0 "#PWR0521" H 1300 2200 50  0001 C CNN
+F 1 "GND" H 1305 2277 50  0000 C CNN
+F 2 "" H 1300 2450 50  0001 C CNN
+F 3 "" H 1300 2450 50  0001 C CNN
+	1    1300 2450
+	1    0    0    -1
+$EndComp
 Wire Notes Line
 	900  1000 8550 1000
@@
 	1350 5750 1600 5750
 Connection ~ 1600 5750
+Wire Wire Line
+	1300 1750 1300 2450
+$Comp
+L power:GND #PWR0522
+U 1 1 5F2C79EA
+P 1650 2450
+F 0 "#PWR0522" H 1650 2200 50  0001 C CNN
+F 1 "GND" H 1655 2277 50  0000 C CNN
+F 2 "" H 1650 2450 50  0001 C CNN
+F 3 "" H 1650 2450 50  0001 C CNN
+	1    1650 2450
+	1    0    0    -1
+$EndComp
+Wire Wire Line
+	1650 2450 1650 2400
+$Comp
+L SMBJ33A-13-F:SMBJ33A-13-F D503
+U 1 1 5F2D9FD2
+P 1650 2400
+F 0 "D503" V 1950 2500 60  0000 R CNN
+F 1 "SMBJ33A-13-F" H 2200 2550 60  0000 R CNN
+F 2 "SMBJ33A-13-F:SMBJ33A-13-F" H 1850 2040 60  0001 C CNN
+F 3 "" H 1650 2400 60  0000 C CNN
+	1    1650 2400
+	0    -1   -1   0
+$EndComp
+Wire Wire Line
+	1300 1550 1650 1550
+Wire Wire Line
+	1650 2000 1650 1550
+Connection ~ 1650 1550
+Wire Wire Line
+	1650 1550 2050 1550
 $EndSCHEMATC

Commit message: ruteado terminado revision basica- 13_07_20
Changed lines of the file:
@@
 	2250 4000 2650 4000
 Wire Wire Line
-	2250 3900 3100 3900
+	2250 3900 2400 3900
 Wire Wire Line
 	3100 3900 3100 4000
@@
 Wire Wire Line
 	1650 1550 2050 1550
+$Comp
+L power:PWR_FLAG #FLG?
+U 1 1 5F1D566B
+P 2400 3900
+F 0 "#FLG?" H 2400 3975 50  0001 C CNN
+F 1 "PWR_FLAG" H 2400 4073 50  0000 C CNN
+F 2 "" H 2400 3900 50  0001 C CNN
+F 3 "~" H 2400 3900 50  0001 C CNN
+	1    2400 3900
+	1    0    0    -1
+$EndComp
+Connection ~ 2400 3900
+Wire Wire Line
+	2400 3900 3100 3900
 $EndSCHEMATC
