File: microcontroladorEsp.sch (KiCad schematic (older format))
At the start: 37 parts, among them J201 USB_B_Micro, J202 Conn_01x02, J203 Conn_01x02, Q201 S8050, Q202 S8050, Q203 2N7002, Q204 2N7002, SW201 SW_Push, SW202 SW_Push, U201 CP2102N-A01-GQFN28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

Commit message: ultima actualizacion antes de iniciar el ruteado, diseño verificado
Parts:
- D202, D203: footprint (none) -> LED_SMD:LED_0805_2012Metric
- SW201, SW202: footprint (none) -> KSR223GLFG:KSR223GLFG
Connections:
- net IO29: no longer names the net of U202.29 (IO5)
- net MISO renamed SPI_MISO
- net MOSI renamed SPI_MOSI
- net SCK renamed SPI_SCK
- no-connect marks 32 -> 36
Other:
- note added: "Boot and Reset SW (SMD)"
- note added: "Microcontrolador ESP32D"
- note removed: "Boot and Reset SW"
- moved on the sheet: C201, C202, C205, C206, C207, R216, SW201, SW202, U202

Commit message: antes de comenzar a rutear
Parts:
- Q201, Q202: footprint Package_TO_SOT_THT:TO-92_Inline -> Package_TO_SOT_SMD:SOT-23
- SW201: value SW_Push -> Reset
- SW202: value SW_Push -> Boot
Connections:
- net GND: no longer J201.6 (Shield)
- no-connect marks 36 -> 37
Changed lines of the file:
@@
 F 0 "Q201" H 2640 6946 50  0000 L CNN
 F 1 "S8050" H 2640 6855 50  0000 L CNN
-F 2 "Package_TO_SOT_THT:TO-92_Inline" H 2650 6825 50  0001 L CIN
+F 2 "Package_TO_SOT_SMD:SOT-23" H 2650 6825 50  0001 L CIN
 F 3 "http://www.unisonic.com.tw/datasheet/S8050.pdf" H 2450 6900 50  0001 L CNN
 	1    2450 6900
@@
 F 0 "Q202" H 2640 7446 50  0000 L CNN
 F 1 "S8050" H 2640 7355 50  0000 L CNN
-F 2 "Package_TO_SOT_THT:TO-92_Inline" H 2650 7325 50  0001 L CIN
+F 2 "Package_TO_SOT_SMD:SOT-23" H 2650 7325 50  0001 L CIN
 F 3 "http://www.unisonic.com.tw/datasheet/S8050.pdf" H 2450 7400 50  0001 L CNN
 	1    2450 7400
@@
 Text Label 1200 7400 2    50   ~ 0
 RTS
-Wire Wire Line
-	1200 6050 1200 6100
-Wire Wire Line
-	1200 6100 1100 6100
-Connection ~ 1100 6100
-Wire Wire Line
-	1100 6100 1100 6050
 NoConn ~ 1500 5850
 Text Label 1500 5750 0    50   ~ 0
@@
 L power:GND #PWR0104
 U 1 1 5ED828EB
-P 1100 6250
-F 0 "#PWR0104" H 1100 6000 50  0001 C CNN
-F 1 "GND" H 1105 6077 50  0000 C CNN
-F 2 "" H 1100 6250 50  0001 C CNN
-F 3 "" H 1100 6250 50  0001 C CNN
-	1    1100 6250
+P 1200 6250
+F 0 "#PWR0104" H 1200 6000 50  0001 C CNN
+F 1 "GND" H 1205 6077 50  0000 C CNN
+F 2 "" H 1200 6250 50  0001 C CNN
+F 3 "" H 1200 6250 50  0001 C CNN
+	1    1200 6250
 	1    0    0    -1
 $EndComp
@@
 	1    0    0    -1
 $EndComp
-Text Label 5050 1500 2    50   ~ 0
+Text Label -2550 3200 2    50   ~ 0
 SW1
 Text Label 6800 1500 2    50   ~ 0
@@
 P 5600 3100
 F 0 "SW201" H 5600 3385 50  0000 C CNN
-F 1 "SW_Push" H 5600 3294 50  0000 C CNN
+F 1 "Reset" H 5600 3294 50  0000 C CNN
 F 2 "KSR223GLFG:KSR223GLFG" H 5600 3300 50  0001 C CNN
 F 3 "~" H 5600 3300 50  0001 C CNN
@@
 P 7500 3150
 F 0 "SW202" H 7500 3435 50  0000 C CNN
-F 1 "SW_Push" H 7500 3344 50  0000 C CNN
+F 1 "Boot" H 7500 3344 50  0000 C CNN
 F 2 "KSR223GLFG:KSR223GLFG" H 7500 3350 50  0001 C CNN
 F 3 "~" H 7500 3350 50  0001 C CNN
@@
 Text Notes 550  550  0    50   ~ 0
 Microcontrolador ESP32D
-Wire Wire Line
-	1100 6100 1100 6250
+NoConn ~ 1100 6050
+Wire Wire Line
+	1200 6050 1200 6250
+Text Label 5050 1500 2    50   ~ 0
+SW1
 $EndSCHEMATC

Commit message: enviado a fabricar
Parts:
- removed D202, D203: LED, LED_SMD:LED_0805_2012Metric, symbol Device:LED
- added J204: Conn_01x04, Connector_PinHeader_2.54mm:PinHeader_1x04_P2.54mm_Vertical, symbol Connector_Generic:Conn_01x04
- added Q205: 2N7002, Package_TO_SOT_SMD:SOT-23, symbol Transistor_FET:2N7002
- added R217: 330K/1%/0603, Resistor_SMD:R_0603_1608Metric, symbol Device:R
- added R218: 10K/1%/0603, Resistor_SMD:R_0603_1608Metric, symbol Device:R
- added R219: 680/1%/0603, Resistor_SMD:R_0603_1608Metric, symbol Device:R
Connections:
- net +5V: now also J204.1 (Pin_1)
- net GND: now also Q205.2 (S), R217.2
- net LED3: now reaches U202.7 (IO35)
- net LED3: now also R217.1, R218.1
- net at R214.1: now also J204.2 (Pin_2)
- net at R215.1: now also J204.4 (Pin_4)
- new net: Q205.1 (G), R218.2
- new net: Q205.3 (D), R219.2
- new net: J204.3 (Pin_3), R219.1
- no-connect marks 37 -> 36
Other:
- moved on the sheet: Q204, R211, R213, R215
Changed lines of the file:
@@
 L Transistor_FET:2N7002 Q204
 U 1 1 5EEFC716
-P 10150 4000
-F 0 "Q204" H 10354 4046 50  0000 L CNN
-F 1 "2N7002" H 10354 3955 50  0000 L CNN
-F 2 "Package_TO_SOT_SMD:SOT-23" H 10350 3925 50  0001 L CIN
-F 3 "https://www.fairchildsemi.com/datasheets/2N/2N7002.pdf" H 10150 4000 50  0001 L CNN
-	1    10150 4000
+P 10150 5200
+F 0 "Q204" H 10354 5246 50  0000 L CNN
+F 1 "2N7002" H 10354 5155 50  0000 L CNN
+F 2 "Package_TO_SOT_SMD:SOT-23" H 10350 5125 50  0001 L CIN
+F 3 "https://www.fairchildsemi.com/datasheets/2N/2N7002.pdf" H 10150 5200 50  0001 L CNN
+	1    10150 5200
 	1    0    0    -1
 $EndComp
@@
 L Device:R R213
 U 1 1 5EF0281A
-P 9700 3850
-F 0 "R213" V 9700 3750 50  0000 L CNN
-F 1 "10K/1%/0603" V 9600 3350 50  0000 L CNN
-F 2 "Resistor_SMD:R_0603_1608Metric" V 9630 3850 50  0001 C CNN
-F 3 "~" H 9700 3850 50  0001 C CNN
-	1    9700 3850
+P 9700 5050
+F 0 "R213" V 9700 4950 50  0000 L CNN
+F 1 "10K/1%/0603" V 9600 4550 50  0000 L CNN
+F 2 "Resistor_SMD:R_0603_1608Metric" V 9630 5050 50  0001 C CNN
+F 3 "~" H 9700 5050 50  0001 C CNN
+	1    9700 5050
 	1    0    0    -1
 $EndComp
@@
 L Device:R R211
 U 1 1 5EF02D6A
-P 9450 3850
-F 0 "R211" V 9450 3750 50  0000 L CNN
-F 1 "330K/1%/0603" V 9350 3350 50  0000 L CNN
-F 2 "Resistor_SMD:R_0603_1608Metric" V 9380 3850 50  0001 C CNN
-F 3 "~" H 9450 3850 50  0001 C CNN
-	1    9450 3850
+P 9450 5050
+F 0 "R211" V 9450 4950 50  0000 L CNN
+F 1 "330K/1%/0603" V 9350 4550 50  0000 L CNN
+F 2 "Resistor_SMD:R_0603_1608Metric" V 9380 5050 50  0001 C CNN
+F 3 "~" H 9450 5050 50  0001 C CNN
+	1    9450 5050
 	1    0    0    -1
 $EndComp
@@
 L Device:R R215
 U 1 1 5EF030F4
-P 10250 3550
-F 0 "R215" V 10250 3450 50  0000 L CNN
-F 1 "680/1%/0603" V 10150 3300 50  0000 L CNN
-F 2 "Resistor_SMD:R_0603_1608Metric" V 10180 3550 50  0001 C CNN
-F 3 "~" H 10250 3550 50  0001 C CNN
-	1    10250 3550
-	1    0    0    -1
-$EndComp
-$Comp
-L Device:LED D203
-U 1 1 5EF07D04
-P 10250 3200
-F 0 "D203" V 10289 3082 50  0000 R CNN
-F 1 "LED" V 10198 3082 50  0000 R CNN
-F 2 "LED_SMD:LED_0805_2012Metric" H 10250 3200 50  0001 C CNN
-F 3 "~" H 10250 3200 50  0001 C CNN
-	1    10250 3200
-	0    -1   -1   0
-$EndComp
-$Comp
-L Device:LED D202
-U 1 1 5EF34631
-P 10250 1250
-F 0 "D202" V 10289 1132 50  0000 R CNN
-F 1 "LED" V 10198 1132 50  0000 R CNN
-F 2 "LED_SMD:LED_0805_2012Metric" H 10250 1250 50  0001 C CNN
-F 3 "~" H 10250 1250 50  0001 C CNN
-	1    10250 1250
-	0    -1   -1   0
+P 10250 4750
+F 0 "R215" V 10250 4650 50  0000 L CNN
+F 1 "680/1%/0603" V 10150 4500 50  0000 L CNN
+F 2 "Resistor_SMD:R_0603_1608Metric" V 10180 4750 50  0001 C CNN
+F 3 "~" H 10250 4750 50  0001 C CNN
+	1    10250 4750
+	1    0    0    -1
 $EndComp
 $Comp
@@
 L power:GND #PWR0219
 U 1 1 5EF3FEC7
-P 10250 4300
-F 0 "#PWR0219" H 10250 4050 50  0001 C CNN
-F 1 "GND" H 10255 4127 50  0000 C CNN
-F 2 "" H 10250 4300 50  0001 C CNN
-F 3 "" H 10250 4300 50  0001 C CNN
-	1    10250 4300
+P 10250 5500
+F 0 "#PWR0219" H 10250 5250 50  0001 C CNN
+F 1 "GND" H 10255 5327 50  0000 C CNN
+F 2 "" H 10250 5500 50  0001 C CNN
+F 3 "" H 10250 5500 50  0001 C CNN
+	1    10250 5500
 	1    0    0    -1
 $EndComp
@@
 L power:GND #PWR0215
 U 1 1 5EF419AE
-P 9450 4300
-F 0 "#PWR0215" H 9450 4050 50  0001 C CNN
-F 1 "GND" H 9455 4127 50  0000 C CNN
-F 2 "" H 9450 4300 50  0001 C CNN
-F 3 "" H 9450 4300 50  0001 C CNN
-	1    9450 4300
-	1    0    0    -1
-$EndComp
-Wire Wire Line
-	10250 1400 10250 1500
+P 9450 5500
+F 0 "#PWR0215" H 9450 5250 50  0001 C CNN
+F 1 "GND" H 9455 5327 50  0000 C CNN
+F 2 "" H 9450 5500 50  0001 C CNN
+F 3 "" H 9450 5500 50  0001 C CNN
+	1    9450 5500
+	1    0    0    -1
+$EndComp
 Wire Wire Line
 	10250 1800 10250 1950
@@
 	9450 2350 9450 2150
 Wire Wire Line
-	9450 4000 9450 4300
-Wire Wire Line
-	9700 4000 9950 4000
-Wire Wire Line
-	10250 3800 10250 3700
-Wire Wire Line
-	10250 4200 10250 4300
-Wire Wire Line
-	10250 3350 10250 3400
-Wire Wire Line
-	9700 3700 9450 3700
-Wire Wire Line
-	9450 3700 9350 3700
-Connection ~ 9450 3700
-$Comp
-L power:+5V #PWR0218
-U 1 1 5EF6C275
-P 10250 2950
-F 0 "#PWR0218" H 10250 2800 50  0001 C CNN
-F 1 "+5V" H 10265 3123 50  0000 C CNN
-F 2 "" H 10250 2950 50  0001 C CNN
-F 3 "" H 10250 2950 50  0001 C CNN
-	1    10250 2950
-	1    0    0    -1
-$EndComp
+	9450 5200 9450 5500
+Wire Wire Line
+	9700 5200 9950 5200
+Wire Wire Line
+	10250 5000 10250 4900
+Wire Wire Line
+	10250 5400 10250 5500
+Wire Wire Line
+	9700 4900 9450 4900
+Wire Wire Line
+	9450 4900 9350 4900
+Connection ~ 9450 4900
 $Comp
 L power:+5V #PWR0216
@@
 Wire Wire Line
 	10250 1000 10250 1100
-Wire Wire Line
-	10250 2950 10250 3050
 Text Label 9350 1850 2    50   ~ 0
 LED1
-Text Label 9350 3700 2    50   ~ 0
+Text Label 9350 4900 2    50   ~ 0
 LED2
 Wire Wire Line
@@
 SW2
 NoConn ~ 2850 3150
-NoConn ~ 2850 3450
 $Comp
 L power:GND #PWR0210
@@
 	1    0    0    -1
 $EndComp
+$Comp
+L Transistor_FET:2N7002 Q205
+U 1 1 5F17E0B4
+P 10150 3550
+F 0 "Q205" H 10354 3596 50  0000 L CNN
+F 1 "2N7002" H 10354 3505 50  0000 L CNN
+F 2 "Package_TO_SOT_SMD:SOT-23" H 10350 3475 50  0001 L CIN
+F 3 "https://www.fairchildsemi.com/datasheets/2N/2N7002.pdf" H 10150 3550 50  0001 L CNN
+	1    10150 3550
+	1    0    0    -1
+$EndComp
+$Comp
+L Device:R R218
+U 1 1 5F17E0BA
+P 9700 3400
+F 0 "R218" V 9700 3300 50  0000 L CNN
+F 1 "10K/1%/0603" V 9600 2900 50  0000 L CNN
+F 2 "Resistor_SMD:R_0603_1608Metric" V 9630 3400 50  0001 C CNN
+F 3 "~" H 9700 3400 50  0001 C CNN
+	1    9700 3400
+	1    0    0    -1
+$EndComp
+$Comp
+L Device:R R217
+U 1 1 5F17E0C0
+P 9450 3400
+F 0 "R217" V 9450 3300 50  0000 L CNN
+F 1 "330K/1%/0603" V 9350 2900 50  0000 L CNN
+F 2 "Resistor_SMD:R_0603_1608Metric" V 9380 3400 50  0001 C CNN
+F 3 "~" H 9450 3400 50  0001 C CNN
+	1    9450 3400
+	1    0    0    -1
+$EndComp
+$Comp
+L Device:R R219
+U 1 1 5F17E0C6
+P 10250 3100
+F 0 "R219" V 10250 3000 50  0000 L CNN
+F 1 "680/1%/0603" V 10150 2850 50  0000 L CNN
+F 2 "Resistor_SMD:R_0603_1608Metric" V 10180 3100 50  0001 C CNN
+F 3 "~" H 10250 3100 50  0001 C CNN
+	1    10250 3100
+	1    0    0    -1
+$EndComp
+$Comp
+L power:GND #PWR0226
+U 1 1 5F17E0D2
+P 10250 3850
+F 0 "#PWR0226" H 10250 3600 50  0001 C CNN
+F 1 "GND" H 10255 3677 50  0000 C CNN
+F 2 "" H 10250 3850 50  0001 C CNN
+F 3 "" H 10250 3850 50  0001 C CNN
+	1    10250 3850
+	1    0    0    -1
+$EndComp
+$Comp
+L power:GND #PWR0203
+U 1 1 5F17E0D8
+P 9450 3850
+F 0 "#PWR0203" H 9450 3600 50  0001 C CNN
+F 1 "GND" H 9455 3677 50  0000 C CNN
+F 2 "" H 9450 3850 50  0001 C CNN
+F 3 "" H 9450 3850 50  0001 C CNN
+	1    9450 3850
+	1    0    0    -1
+$EndComp
+Wire Wire Line
+	9450 3550 9450 3850
+Wire Wire Line
+	9700 3550 9950 3550
+Wire Wire Line
+	10250 3350 10250 3250
+Wire Wire Line
+	10250 3750 10250 3850
+Wire Wire Line
+	10250 2900 10250 2950
+Wire Wire Line
+	9700 3250 9450 3250
+Wire Wire Line
+	9450 3250 9350 3250
+Connection ~ 9450 3250
+Text Label 9350 3250 2    50   ~ 0
+LED3
+Wire Wire Line
+	2850 3450 3250 3450
+Text Label 3250 3450 0    50   ~ 0
+LED3
+$Comp
+L Connector_Generic:Conn_01x04 J204
+U 1 1 5F19AE79
+P 11000 1200
+F 0 "J204" H 11080 1192 50  0000 L CNN
+F 1 "Conn_01x04" H 11080 1101 50  0000 L CNN
+F 2 "Connector_PinHeader_2.54mm:PinHeader_1x04_P2.54mm_Vertical" H 11000 1200 50  0001 C CNN
+F 3 "~" H 11000 1200 50  0001 C CNN
+	1    11000 1200
+	1    0    0    -1
+$EndComp
+Wire Wire Line
+	10800 1100 10250 1100
+Wire Wire Line
+	10250 1200 10800 1200
+Wire Wire Line
+	10250 1200 10250 1500
+Wire Wire Line
+	10700 1300 10800 1300
+Wire Wire Line
+	10800 1400 10750 1400
+Wire Wire Line
+	10250 4450 10250 4600
+Wire Wire Line
+	10250 2900 10700 2900
+Wire Wire Line
+	10700 2900 10700 1300
+Wire Wire Line
+	10750 1400 10750 4450
+Wire Wire Line
+	10750 4450 10250 4450
 $EndSCHEMATC
